File: NRF52832/NRF52832 v01.sch (KiCad schematic (older format))
At the start: 17 parts, among them U1 NRF52832_QFN48, Y1 32.768kHz, Y2 32MHz

Commit message: Some little changes and a .net
Parts:
- removed Y2: 32MHz, symbol Crystal
- added Y2: Crystal_GND24, Crystals:Crystal_SMD_3225-4pin_3.2x2.5mm_HandSoldering, symbol Crystal_GND24
- C1, C10, C11, C2, C3, C4, C5, C6, C7, C8, C9: footprint (none) -> Capacitors_SMD:C_0805_HandSoldering
- L1, L2, L3: footprint (none) -> Inductors:Inductor_Taiyo-Yuden_NR-20xx_HandSoldering
- U1: footprint (none) -> Housings_DFN_QFN:UQFN-48-1EP_6x6mm_Pitch0.4mm
- Y1: footprint (none) -> Crystals:Crystal_SMD_3215-2pin_3.2x1.5mm
Connections:
- net at U1.1 (DEC1): now also C4.2
- net at U1.34 (XC1): now also Y2.1; no longer C10.2
- net at U1.35 (XC2): now also Y2.3; no longer C9.2
- new net: C9.2, Y2.4
- new net: C10.2, Y2.2
Other:
- moved on the sheet: C10, C9
